Commit message: captures

File: 2. Kinematics/Lab/urdf_model/urdf/robot_arm.urdf (robot description, URDF)
Before this commit: robot visual, 5 links, 4 joints
Joints:
- joint cyl1_cyl2: axis 0 1 0 -> 0 -1 0

Commit message: correction angles

File: 2. Kinematics/Lab/urdf_model/urdf/robot_arm.urdf (robot description, URDF)
Before this commit: robot visual, 5 links, 4 joints
Links:
- link base_link: geometry visual cylinder length=0.05 radius=0.1
- link cyl1: geometry visual cylinder length=0.45 radius=0.05
Joints:
- joint base_cyl1: origin xyz=0 0 0 -> xyz=0 0 0.05
- joint cyl1_cyl2: origin xyz=0 -0.1 0.5 -> xyz=0 -0.1 0.4 rpy=0 1.57075 0
- joint cyl2_cyl3: origin xyz=0.35 0.1 0 -> xyz=0 0.1 0.35
- joint cyl3_box: axis 1 0 0 -> 0 0 1; origin xyz=0.35 0 0 -> xyz=0 0 0.35
